Commit message: rename dynaarm_control xacro macro to dynaarm

File: duatic_dynaarm_driver/duatic_dynaarm_driver/urdf/dynaarm.urdf.xacro (robot description, xacro)
@@ -23,5 +23,5 @@
 <!-- This macro combines the actual description together with the ros2control plugin description-->
 <robot name="dynaarm" xmlns:xacro="http://www.ros.org/wiki/xacro">
-    <xacro:macro name="dynaarm_control"
+    <xacro:macro name="dynaarm"
     params="tf_prefix parent_link collision:='simple' dof mode ethercat_bus drive_order:='' start_in_freeze_mode:=false drive_parameter_folder:='' covers version *origin">
         <xacro:include filename="$(find duatic_dynaarm_description)/urdf/dynaarm.urdf.xacro" />
@@ -33,5 +33,5 @@
         <xacro:property name="ethercat_addresses" value="${xacro.load_yaml(drive_order_file)}"/>
         <!-- Create the instance of the actual description (what you see in rviz)-->
-        <xacro:dynaarm
+        <xacro:dynaarm_description
                 tf_prefix="${tf_prefix}"
                 parent_link="${parent_link}"
@@ -41,5 +41,5 @@
                 version="${version}">
             <xacro:insert_block name="origin" />
-        </xacro:dynaarm>
+        </xacro:dynaarm_description>
         <!-- Creatte the ros2control part-->
         <xacro:dynaarm_ros2_control tf_prefix="${tf_prefix}"
